File: Coulomb_Counter.kicad_pcb (KiCad board)
At the start: 2 copper layers, 29.8 x 15.2 mm, 18 parts, among them P1 JST, P2 IN, P3 OUT, P4 CONN_01X06, U1 LTC4150

Commit message: Final design
Parts:
- added U2: EE_Logo, EE_Logo:Logo_8, B.Cu at (160.0, 62.7)
- added U3: MountingHole, Connect:1pin, F.Cu at (163.3, 56.9)
- added U4: MountingHole, Connect:1pin, F.Cu at (163.3, 68.8)
Routing:
- net Net-(JP3-Pad1): track 18.1 -> 17.2 mm
- added copper zone on B.Cu, net GND
- added copper zone on F.Cu, net Net-(C1-Pad1)
Other:
- outline, holes or cut-outs redrawn
- board text added: "Coulomb Counter"
- board text added: "ExploreEmbedded.com"
