File: _saved_Coulomb_Counter.sch (KiCad schematic (older format))
At the start: 18 parts, among them P1 JST, P2 IN, P3 OUT, P4 CONN_01X06, U1 LTC4150

Commit message: Final design
Parts:
- added U2: EE_Logo, EE_Logo:Logo_8, symbol EE_Logo
- added U3, U4: MountingHole, Connect:1pin, symbol MountingHole
Changed lines of the file:
@@
 LIBS:contrib
 LIBS:valves
+LIBS:ExploreM3-cache
 LIBS:Coulomb_Counter-cache
 EELAYER 25 0
@@
 	7550 2350 7550 2250
 Connection ~ 7550 2250
+$Comp
+L EE_Logo U2
+U 1 1 58AD098D
+P 8550 2850
+F 0 "U2" H 8550 2700 40  0000 C CNN
+F 1 "EE_Logo" H 8550 2760 40  0000 C CNN
+F 2 "EE_Logo:Logo_8" H 8550 2850 40  0001 C CNN
+F 3 "" H 8550 2850 40  0000 C CNN
+	1    8550 2850
+	1    0    0    -1
+$EndComp
+$Comp
+L MountingHole U3
+U 1 1 58AD0A3E
+P 9050 2800
+F 0 "U3" H 9050 2650 40  0000 C CNN
+F 1 "MountingHole" H 9050 2700 40  0000 C CNN
+F 2 "Connect:1pin" H 9050 2800 40  0001 C CNN
+F 3 "" H 9050 2800 40  0000 C CNN
+	1    9050 2800
+	1    0    0    -1
+$EndComp
+$Comp
+L MountingHole U4
+U 1 1 58AD0BD7
+P 9600 2800
+F 0 "U4" H 9600 2650 40  0000 C CNN
+F 1 "MountingHole" H 9600 2700 40  0000 C CNN
+F 2 "Connect:1pin" H 9600 2800 40  0001 C CNN
+F 3 "" H 9600 2800 40  0000 C CNN
+	1    9600 2800
+	1    0    0    -1
+$EndComp
 $EndSCHEMATC
